File: pedal.kicad_sch (KiCad schematic)
At the start: 46 parts, among them J1 Conn_01x03_Socket, J2 Conn_01x01_Pin, J3 Conn_01x01_Pin, J4 Conn_01x01_Pin, J5 Conn_01x01_Pin, J6 Conn_01x02_Socket, SW1 EG5498-ND, SW2 SW_SPDT, SW3 EG5498-ND, T1 142B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

Commit message: Add files via upload
Connections:
- net at RV3.1, SW3.1 (A): now also SW3.6 (C); no longer SW3.4 (A)
Changed lines of the file:
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@@
     )
   )
-  (symbol (lib_id "Switch:SW_DPDT_x2") (at 220.98 132.08 0) (unit 2)
+  (symbol (lib_id "Switch:SW_DPDT_x2") (at 220.98 132.08 0) (mirror x) (unit 2)
     (in_bom yes) (on_board yes) (dnp no)
-    (property "Reference" "SW3" (at 220.98 137.16 0)
+    (property "Reference" "SW3" (at 220.98 138.43 0)
       (effects (font (size 1.27 1.27)))
     )
-    (property "Value" "	\nEG5498-ND" (at 220.98 138.43 0)
+    (property "Value" "	\nEG5498-ND" (at 222.25 139.7 0)
       (effects (font (size 1.27 1.27)))
     )

Commit message: Add files via upload
Fixed some small errors.
Connections:
- net GND: now also BT1.2 (-), C2.2, C7.2, C8.2, R3.2, R6.2, U1.11 (V-)
Other:
- moved on the sheet: BT1, C2, C7, C8, D1, D2, R2, R3, R6, SW2, U1E

Commit message: Add files via upload
Parts:
- added J7, J8: Conn_01x01_Pin, Connector_PinHeader_2.00mm:PinHeader_1x01_P2.00mm_Vertical, symbol Connector:Conn_01x01_Pin
Connections:
- net Bypass: now also J8.1 (Pin_1)
- net OUT: now also J7.1 (Pin_1)
Changed lines of the file:
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@@
   (junction (at 77.47 87.63) (diameter 0) (color 0 0 0 0)
   )
+  (junction (at 45.72 115.57) (diameter 0) (color 0 0 0 0)
+  )
   (junction (at 80.01 29.21) (diameter 0) (color 0 0 0 0)
   )
@@
   )
   (junction (at 120.65 176.53) (diameter 0) (color 0 0 0 0)
+  )
+  (junction (at 73.66 180.34) (diameter 0) (color 0 0 0 0)
   )
   (junction (at 95.25 96.52) (diameter 0) (color 0 0 0 0)
@@
     (stroke (width 0) (type default))
   )
+  (wire (pts (xy 45.72 115.57) (xy 43.18 115.57))
+    (stroke (width 0) (type default))
+  )
   (wire (pts (xy 204.47 142.24) (xy 207.01 142.24))
     (stroke (width 0) (type default))
@@
   )
   (wire (pts (xy 123.19 29.21) (xy 123.19 26.67))
+    (stroke (width 0) (type default))
+  )
+  (wire (pts (xy 49.53 115.57) (xy 45.72 115.57))
     (stroke (width 0) (type default))
   )
@@
     )
   )
-  (global_label "Bypass" (shape input) (at 43.18 115.57 0) (fields_autoplaced)
+  (global_label "Bypass" (shape input) (at 49.53 115.57 0) (fields_autoplaced)
     (effects (font (size 1.27 1.27)) (justify left))
-    (property "Intersheetrefs" "${INTERSHEET_REFS}" (at 52.757 115.57 0)
+    (property "Intersheetrefs" "${INTERSHEET_REFS}" (at 59.107 115.57 0)
       (effects (font (size 1.27 1.27)) (justify left) hide)
     )
@@
         (path "/602b8f86-9d3e-48c5-a967-fc9f56706963"
           (reference "#PWR011") (unit 1)
+        )
+      )
+    )
+  )
+  (symbol (lib_id "Connector:Conn_01x01_Pin") (at 73.66 175.26 270) (unit 1)
+    (in_bom yes) (on_board yes) (dnp no)
+    (property "Reference" "J7" (at 78.74 175.895 0)
+      (effects (font (size 1.27 1.27)))
+    )
+    (property "Value" "Conn_01x01_Pin" (at 73.66 165.1 0)
+      (effects (font (size 1.27 1.27)))
+    )
+    (property "Footprint" "Connector_PinHeader_2.00mm:PinHeader_1x01_P2.00mm_Vertical" (at 73.66 175.26 0)
+      (effects (font (size 1.27 1.27)) hide)
+    )
+    (property "Datasheet" "~" (at 73.66 175.26 0)
+      (effects (font (size 1.27 1.27)) hide)
+    )
+    (pin "1")
+    (instances
+      (project "pedal"
+        (path "/602b8f86-9d3e-48c5-a967-fc9f56706963"
+          (reference "J7") (unit 1)
         )
       )
@@
         )
       )
+    )
+  )
+  (symbol (lib_id "Connector:Conn_01x01_Pin") (at 45.72 120.65 90) (unit 1)
+    (in_bom yes) (on_board yes) (dnp no)
+    (property "Reference" "J8" (at 46.99 118.745 90)
+      (effects (font (size 1.27 1.27)) (justify right))
+    )
+    (property "Value" "Conn_01x01_Pin" (at 40.64 121.92 90)
+      (effects (font (size 1.27 1.27)) (justify right))
+    )
+    (property "Footprint" "Connector_PinHeader_2.00mm:PinHeader_1x01_P2.00mm_Vertical" (at 45.72 120.65 0)
+      (effects (font (size 1.27 1.27)) hide)
+    )
+    (property "Datasheet" "~" (at 45.72 120.65 0)
+      (effects (font (size 1.27 1.27)) hide)
+    )
+    (pin "1")
+    (instances
+      (project "pedal"
+        (path "/602b8f86-9d3e-48c5-a967-fc9f56706963"
+          (reference "J8") (unit 1)
+        )
+      )
